File: files/pcb/splitbk/splitbk.kicad_pcb (KiCad board)
At the start: 2 copper layers, 3.8 x 3 mm, 186 parts, among them J1 L_TRRS, J2 L_TRRS, SW1 CherryMX, SW10 CherryMX, SW11 CherryMX, SW12 CherryMX, SW13 CherryMX, SW14 CherryMX, SW15 CherryMX, SW16 CherryMX, SW17 CherryMX, SW18 CherryMX, SW19 CherryMX, SW2 CherryMX, SW20 CherryMX, SW21 CherryMX, SW22 CherryMX, SW23 CherryMX, SW24 CherryMX, SW25 CherryMX, SW26 CherryMX, SW27 CherryMX, SW28 CherryMX, SW29 CherryMX, SW3 CherryMX, SW30 CherryMX, SW31 CherryMX, SW32 CherryMX, SW33 CherryMX, SW34 CherryMX, SW35 CherryMX, SW36 CherryMX, SW37 CherryMX, SW38 CherryMX, SW39 CherryMX, SW4 CherryMX, SW40 CherryMX, SW41 CherryMX, SW42 RotaryEncoder, SW43 CherryMX, SW44 CherryMX, SW45 CherryMX, SW46 CherryMX, SW47 CherryMX, SW48 CherryMX, SW49 CherryMX, SW5 CherryMX, SW50 CherryMX, SW51 CherryMX, SW52 CherryMX, SW53 RotaryEncoder, SW54 CherryMX, SW55 CherryMX, SW56 CherryMX, SW57 CherryMX, SW58 CherryMX, SW59 CherryMX, SW6 CherryMX, SW60 CherryMX, SW61 CherryMX, SW7 CherryMX, SW8 CherryMX, SW9 CherryMX, U1 Pico, U2 Pico

Commit message: All rows wired, Moving onto rightside LED placement
Parts:
- D44, D45, D46, D47, D48, D49, D50, D51, D52, D53, D54, D55, D56, D57, D58, D59: moved to B.Cu
- moved D51 276.4 mm to (264.8, 95.2), turned to 90 degrees
- moved D56 263.6 mm to (276.8, 114.3), turned to 90 degrees
- moved D52 257.6 mm to (283.8, 95.2), turned to 90 degrees
- moved D44 246.4 mm to (272.4, 76.2), turned to 90 degrees
- moved D45 234.8 mm to (291.5, 76.2), turned to 90 degrees
- moved D53 228.0 mm to (302.9, 95.2), turned to 90 degrees
- moved D46 222.3 mm to (310.5, 76.2), turned to 90 degrees
- moved D57 215.4 mm to (314.9, 114.3), turned to 90 degrees
- moved D54 210.6 mm to (321.9, 95.2), turned to 90 degrees
- moved D47 206.1 mm to (329.6, 76.2), turned to 90 degrees
- moved D58 201.2 mm to (341.0, 114.3), turned to 90 degrees
- moved D55 199.3 mm to (341.0, 95.2), turned to 90 degrees
- moved D48 192.6 mm to (348.6, 76.4), turned to 90 degrees
- moved D49 175.7 mm to (367.7, 76.4), turned to 90 degrees
- moved D59 164.1 mm to (376.8, 114.3), turned to 90 degrees
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Routing:
- net R_R4: track 0.00 -> 191.7 mm
- net R_R2: track 0.00 -> 174.6 mm
- net R_R3: track 0.00 -> 153.2 mm
- net R_R1: track 117.8 -> 166.3 mm
- net Net-(D49-A): track 0.00 -> 4.29 mm
- net Net-(D48-A): track 0.00 -> 4.29 mm
- net Net-(D59-A): track 0.00 -> 4.13 mm
- net Net-(D57-A): track 0.00 -> 4.13 mm
- net Net-(D56-A): track 0.00 -> 4.13 mm
- net Net-(D58-A): track 0.00 -> 4.09 mm
- net Net-(D55-A): track 0.00 -> 4.09 mm
- net Net-(D54-A): track 0.00 -> 4.09 mm
- net Net-(D52-A): track 0.00 -> 4.09 mm
- net Net-(D51-A): track 0.00 -> 4.09 mm
- net Net-(D47-A): track 0.00 -> 4.09 mm
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
Commit message: PCB Routing Completed
Parts:
- removed D65.5: WS2812B, footprints:SK6812-MINI-E
- D35.5, D36.5, D37.5, D38.5, D39.5, D40.5, D41.5, D42.5, D43.5, D44.5, D45.5, D46.5, D47.5, D48.5, D49.5, D50.5, D51.5, D52.5, D53.5, D54.5, D55.5, D56.5, D57.5, D58.5, D59.5, D60.5, D61.5, D62.5, D63.5, D64.5: moved to B.Cu
- moved D55.5 355.2 mm to (257.2, 100.4), turned to 180 degrees
- moved D41.5 354.7 mm to (261.9, 62.3), turned to 180 degrees
- moved D48.5 349.6 mm to (264.8, 81.3), turned to 180 degrees
- moved D61.5 342.4 mm to (268.6, 119.4), turned to 180 degrees
- moved D35.5 342.1 mm to (257.2, 43.2), turned to 180 degrees
- moved D36.5 332.7 mm to (276.4, 43.2), turned to 180 degrees
- moved D56.5 317.9 mm to (276.2, 100.4), turned to 180 degrees
- moved D42.5 315.7 mm to (281.0, 62.3), turned to 180 degrees
- moved D37.5 311.5 mm to (295.3, 43.2), turned to 180 degrees
- moved D49.5 309.8 mm to (283.8, 81.3), turned to 180 degrees
- moved D43.5 306.2 mm to (300.0, 62.3), turned to 180 degrees
- moved D38.5 305.3 mm to (314.3, 43.2), turned to 180 degrees
- moved D57.5 302.6 mm to (295.3, 100.4), turned to 180 degrees
- moved D50.5 292.0 mm to (302.9, 81.3), turned to 180 degrees
- moved D58.5 287.5 mm to (314.3, 100.4), turned to 180 degrees
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Connections:
- D35.5 pad 4: R_LED -> R_RGB
- D64.5 pad 2: Net-(D64.5-DOUT) -> unconnected-(D64.5-DOUT-Pad2)
- SW49 pad 1: unconnected-(SW49-Pad1) -> R_C8
- U2 pad 14: unconnected-(U2-GPIO10-Pad14) -> R_C10
- U2 pad 15: unconnected-(U2-GPIO11-Pad15) -> R_C11
- U2 pad 16: unconnected-(U2-GPIO12-Pad16) -> R_C12
- U2 pad 17: unconnected-(U2-GPIO13-Pad17) -> R_C13
Routing:
- net R_VBUS: track 0.00 -> 780.1 mm, vias 0 -> 8
- net R_C11: track 0.00 -> 278.6 mm, vias 0 -> 5
- net R_C12: track 0.00 -> 255.1 mm, vias 0 -> 3
- net R_C13: track 0.00 -> 233.0 mm, vias 0 -> 2
- net R_C10: track 0.00 -> 227.0 mm, vias 0 -> 5
- net R_ECB: track 0.00 -> 200.1 mm, vias 0 -> 1
- net R_C9: track 0.00 -> 198.0 mm, vias 0 -> 5
- net R_ECA: track 0.00 -> 193.2 mm, vias 0 -> 1
- net R_C8: track 0.00 -> 171.0 mm, vias 0 -> 5
- net Net-(D54.5-DOUT): track 0.00 -> 148.8 mm, vias 0 -> 2
- net Net-(D47.5-DOUT): track 0.00 -> 139.4 mm, vias 0 -> 2
- net Net-(D60.5-DOUT): track 0.00 -> 134.4 mm, vias 0 -> 2
- net Net-(D40.5-DOUT): track 0.00 -> 125.8 mm, vias 0 -> 2
- net R_C7: track 0.00 -> 105.1 mm, vias 0 -> 4
- net R_RGB: track 0.00 -> 58.5 mm, vias 0 -> 4
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- added copper zone on B.Cu, net GND
- added copper zone on F.Cu, net GND
Other:
- board size 3.8 x 3 mm -> 360.7 x 102.2 mm
