File: files/pcb/splitbk/splitbk.kicad_sch (KiCad schematic)
At the start: 186 parts, among them J1 L_TRRS, J2 L_TRRS, SW1 CherryMX, SW10 CherryMX, SW11 CherryMX, SW12 CherryMX, SW13 CherryMX, SW14 CherryMX, SW15 CherryMX, SW16 CherryMX, SW17 CherryMX, SW18 CherryMX, SW19 CherryMX, SW2 CherryMX, SW20 CherryMX, SW21 CherryMX, SW22 CherryMX, SW23 CherryMX, SW24 CherryMX, SW25 CherryMX, SW26 CherryMX, SW27 CherryMX, SW28 CherryMX, SW29 CherryMX, SW3 CherryMX, SW30 CherryMX, SW31 CherryMX, SW32 CherryMX, SW33 CherryMX, SW34 CherryMX, SW35 CherryMX, SW36 CherryMX, SW37 CherryMX, SW38 CherryMX, SW39 CherryMX, SW4 CherryMX, SW40 CherryMX, SW41 CherryMX, SW42 RotaryEncoder, SW43 CherryMX, SW44 CherryMX, SW45 CherryMX, SW46 CherryMX, SW47 CherryMX, SW48 CherryMX, SW49 CherryMX, SW5 CherryMX, SW50 CherryMX, SW51 CherryMX, SW52 CherryMX, SW53 RotaryEncoder, SW54 CherryMX, SW55 CherryMX, SW56 CherryMX, SW57 CherryMX, SW58 CherryMX, SW59 CherryMX, SW6 CherryMX, SW60 CherryMX, SW61 CherryMX, SW7 CherryMX, SW8 CherryMX, SW9 CherryMX, U1 Pico, U2 Pico

Commit message: All rows wired, Moving onto rightside LED placement
Parts:
- removed D65.5: WS2812B, footprints:SK6812-MINI-E, symbol LED:WS2812B
Connections:
- net R_C8: now also SW49.1
Changed lines of the file:
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@@
 	)
 	(junction
+		(at 721.36 243.84)
+		(diameter 0)
+		(color 0 0 0 0)
+	)
+	(junction
 		(at 943.61 204.47)
 		(diameter 0)
@@
 	)
 	(junction
-		(at 1045.21 276.86)
-		(diameter 0)
-		(color 0 0 0 0)
-	)
-	(junction
 		(at 1043.94 260.35)
 		(diameter 0)
@@
 	)
 	(junction
-		(at 1070.61 292.1)
-		(diameter 0)
-		(color 0 0 0 0)
-	)
-	(junction
 		(at 207.01 215.9)
 		(diameter 0)
@@
 	)
 	(no_connect
-		(at 1078.23 284.48)
+		(at 1052.83 284.48)
 	)
 	(wire
@@
 	(wire
 		(pts
+			(xy 721.36 243.84) (xy 727.71 243.84)
+		)
+		(stroke
+			(width 0)
+			(type default)
+		)
+	)
+	(wire
+		(pts
 			(xy 412.75 166.37) (xy 438.15 166.37)
 		)
@@
 	(wire
 		(pts
-			(xy 1052.83 284.48) (xy 1062.99 284.48)
-		)
-		(stroke
-			(width 0)
-			(type default)
-		)
-	)
-	(wire
-		(pts
 			(xy 76.2 241.3) (xy 156.21 241.3)
 		)
@@
 	(wire
 		(pts
-			(xy 721.36 269.24) (xy 721.36 218.44)
+			(xy 721.36 269.24) (xy 721.36 243.84)
 		)
 		(stroke
@@
 	(wire
 		(pts
+			(xy 721.36 243.84) (xy 721.36 218.44)
+		)
+		(stroke
+			(width 0)
+			(type default)
+		)
+	)
+	(wire
+		(pts
 			(xy 910.59 224.79) (xy 910.59 210.82)
 		)
@@
 	(wire
 		(pts
-			(xy 1045.21 276.86) (xy 1070.61 276.86)
-		)
-		(stroke
-			(width 0)
-			(type default)
-		)
-	)
-	(wire
-		(pts
 			(xy 165.1 182.88) (xy 165.1 208.28)
 		)
@@
 	(wire
 		(pts
-			(xy 1045.21 292.1) (xy 1070.61 292.1)
-		)
-		(stroke
-			(width 0)
-			(type default)
-		)
-	)
-	(wire
-		(pts
 			(xy 918.21 161.29) (xy 943.61 161.29)
 		)
@@
 	)
 	(symbol
-		(lib_id "power:GND")
-		(at 1070.61 292.1 0)
-		(unit 1)
-		(exclude_from_sim no)
-		(in_bom yes)
-		(on_board yes)
-		(dnp no)
-		(fields_autoplaced yes)
-		(property "Reference" "#PWR7"
-			(at 1070.61 298.45 0)
-			(effects
-				(font
-					(size 1.27 1.27)
-				)
-				(hide yes)
-			)
-		)
-		(property "Value" "GND"
-			(at 1070.61 297.18 0)
-			(effects
-				(font
-					(size 1.27 1.27)
-				)
-			)
-		)
-		(property "Footprint" ""
-			(at 1070.61 292.1 0)
-			(effects
-				(font
-					(size 1.27 1.27)
-				)
-				(hide yes)
-			)
-		)
-		(property "Datasheet" ""
-			(at 1070.61 292.1 0)
-			(effects
-				(font
-					(size 1.27 1.27)
-				)
-				(hide yes)
-			)
-		)
-		(property "Description" "Power symbol creates a global label with name \"GND\" , ground"
-			(at 1070.61 292.1 0)
-			(effects
-				(font
-					(size 1.27 1.27)
-				)
-				(hide yes)
-			)
-		)
-		(pin "1"
-		)
-		(instances
-			(project "splitbk"
-				(path "/8fd27b71-1cc7-4b76-b115-4e496c9b4baa"
-					(reference "#PWR7")
-					(unit 1)
-				)
-			)
-		)
-	)
-	(symbol
 		(lib_id "CherryMX:CherryMX")
 		(at 100.33 182.88 0)
@@
 	)
 	(symbol
+		(lib_id "power:GND")
+		(at 1045.21 292.1 0)
+		(unit 1)
+		(exclude_from_sim no)
+		(in_bom yes)
+		(on_board yes)
+		(dnp no)
+		(fields_autoplaced yes)
+		(property "Reference" "#PWR7"
+			(at 1045.21 298.45 0)
+			(effects
+				(font
+					(size 1.27 1.27)
+				)
+				(hide yes)
+			)
+		)
+		(property "Value" "GND"
+			(at 1045.21 297.18 0)
+			(effects
+				(font
+					(size 1.27 1.27)
+				)
+			)
+		)
+		(property "Footprint" ""
+			(at 1045.21 292.1 0)
+			(effects
+				(font
+					(size 1.27 1.27)
+				)
+				(hide yes)
+			)
+		)
+		(property "Datasheet" ""
+			(at 1045.21 292.1 0)
+			(effects
+				(font
+					(size 1.27 1.27)
+				)
+				(hide yes)
+			)
+		)
+		(property "Description" "Power symbol creates a global label with name \"GND\" , ground"
+			(at 1045.21 292.1 0)
+			(effects
+				(font
+					(size 1.27 1.27)
+				)
+				(hide yes)
+			)
+		)
+		(pin "1"
+		)
+		(instances
+			(project "splitbk"
+				(path "/8fd27b71-1cc7-4b76-b115-4e496c9b4baa"
+					(reference "#PWR7")
+					(unit 1)
+				)
+			)
+		)
+	)
+	(symbol
 		(lib_id "Device:D")
 		(at 181.61 237.49 90)
@@
 					(unit 1)
 				)
-			)
-		)
-	)
-	(symbol
-		(lib_id "LED:WS2812B")
-		(at 1070.61 284.48 0)
-		(unit 1)
-		(exclude_from_sim no)
-		(in_bom yes)
-		(on_board yes)
-		(dnp no)
-		(fields_autoplaced yes)
-		(property "Reference" "D65.5"
-			(at 1082.04 278.1614 0)
-			(effects
-				(font
-					(size 1.27 1.27)
-				)
-			)
-		)
-		(property "Value" "WS2812B"
-			(at 1082.04 280.7014 0)
-			(effects
-				(font
-					(size 1.27 1.27)
-				)
-			)
-		)
-		(property "Footprint" "footprints:SK6812-MINI-E"
-			(at 1071.88 292.1 0)
-			(effects
-				(font
-					(size 1.27 1.27)
-				)
-				(justify left top)
-				(hide yes)
-			)
-		)
-		(property "Datasheet" "https://cdn-shop.adafruit.com/datasheets/WS2812B.pdf"
-			(at 1073.15 294.005 0)
-			(effects
-				(font
-					(size 1.27 1.27)
-				)
-				(justify left top)
-				(hide yes)
-			)
-		)
-		(property "Description" "RGB LED with integrated controller"
-			(at 1070.61 284.48 0)
-			(effects
-				(font
-					(size 1.27 1.27)
-				)
-				(hide yes)
-			)
-		)
-		(pin "2"
-		)
-		(pin "1"
-		)
-		(pin "3"
-		)
-		(pin "4"
-		)
-		(instances
-			(project "splitbk"
-				(path "/8fd27b71-1cc7-4b76-b115-4e496c9b4baa"
-					(reference "D65.5")
-					(unit 1)
-				)

Commit message: PCB Routing Completed
Connections:
- net R_LED is gone; now on net R_RGB: D35.5.4 (DIN)
- net R_C10: now also U2.14 (GPIO10)
- net R_C11: now also U2.15 (GPIO11)
- net R_C12: now also U2.16 (GPIO12)
- net R_C13: now also U2.17 (GPIO13)
- no-connect marks 2 -> 36
Changed lines of the file:
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@@
 	)
 	(no_connect
+		(at 313.69 123.19)
+	)
+	(no_connect
+		(at 298.45 130.81)
+	)
+	(no_connect
+		(at 313.69 80.01)
+	)
+	(no_connect
+		(at 313.69 97.79)
+	)
+	(no_connect
+		(at 313.69 115.57)
+	)
+	(no_connect
+		(at 313.69 100.33)
+	)
+	(no_connect
 		(at 394.97 270.51)
 	)
 	(no_connect
+		(at 313.69 105.41)
+	)
+	(no_connect
+		(at 313.69 85.09)
+	)
+	(no_connect
+		(at 278.13 123.19)
+	)
+	(no_connect
+		(at 313.69 125.73)
+	)
+	(no_connect
+		(at 920.75 107.95)
+	)
+	(no_connect
+		(at 900.43 140.97)
+	)
+	(no_connect
+		(at 920.75 133.35)
+	)
+	(no_connect
+		(at 920.75 113.03)
+	)
+	(no_connect
 		(at 1052.83 284.48)
 	)
+	(no_connect
+		(at 313.69 118.11)
+	)
+	(no_connect
+		(at 920.75 115.57)
+	)
+	(no_connect
+		(at 920.75 135.89)
+	)
+	(no_connect
+		(at 920.75 97.79)
+	)
+	(no_connect
+		(at 313.69 95.25)
+	)
+	(no_connect
+		(at 920.75 102.87)
+	)
+	(no_connect
+		(at 920.75 100.33)
+	)
+	(no_connect
+		(at 905.51 140.97)
+	)
+	(no_connect
+		(at 920.75 128.27)
+	)
+	(no_connect
+		(at 920.75 110.49)
+	)
+	(no_connect
+		(at 313.69 90.17)
+	)
+	(no_connect
+		(at 920.75 125.73)
+	)
+	(no_connect
+		(at 920.75 95.25)
+	)
+	(no_connect
+		(at 313.69 92.71)
+	)
+	(no_connect
+		(at 313.69 102.87)
+	)
+	(no_connect
+		(at 885.19 133.35)
+	)
+	(no_connect
+		(at 920.75 90.17)
+	)
+	(no_connect
+		(at 313.69 87.63)
+	)
+	(no_connect
+		(at 293.37 130.81)
+	)
+	(no_connect
+		(at 920.75 105.41)
+	)
 	(wire
 		(pts
@@
 	(global_label "R_C10"
 		(shape input)
-		(at 886.46 120.65 180)
+		(at 885.19 120.65 180)
 		(fields_autoplaced yes)
 		(effects
@@
 		)
 		(property "Intersheetrefs" "${INTERSHEET_REFS}"
-			(at 877.5482 120.65 0)
+			(at 876.2782 120.65 0)
 			(effects
 				(font
@@
 	(global_label "R_C12"
 		(shape input)
-		(at 886.46 125.73 180)
+		(at 885.19 125.73 180)
 		(fields_autoplaced yes)
 		(effects
@@
 		)
 		(property "Intersheetrefs" "${INTERSHEET_REFS}"
-			(at 877.5482 125.73 0)
+			(at 876.2782 125.73 0)
 			(effects
 				(font
@@
 		)
 	)
-	(global_label "R_LED"
+	(global_label "R_RGB"
 		(shape input)
 		(at 910.59 168.91 180)
@@
 		)
 		(property "Intersheetrefs" "${INTERSHEET_REFS}"
-			(at 901.9201 168.91 0)
+			(at 901.5572 168.91 0)
 			(effects
 				(font
@@
 	(global_label "R_C11"
 		(shape input)
-		(at 886.46 123.19 180)
+		(at 885.19 123.19 180)
 		(fields_autoplaced yes)
 		(effects
@@
 		)
 		(property "Intersheetrefs" "${INTERSHEET_REFS}"
-			(at 877.5482 123.19 0)
+			(at 876.2782 123.19 0)
 			(effects
 				(font
@@
 	(global_label "R_C13"
 		(shape input)
-		(at 886.46 128.27 180)
+		(at 885.19 128.27 180)
 		(fields_autoplaced yes)
 		(effects
@@
 		)
 		(property "Intersheetrefs" "${INTERSHEET_REFS}"
-			(at 877.5482 128.27 0)
+			(at 876.2782 128.27 0)
 			(effects
 				(font
