File: split-kola/pcb/split-kola/split-kola.kicad_pcb (KiCad board)
At the start: 2 copper layers, 360.4 x 103.2 mm, 185 parts, among them J1 L_TRRS, J2 L_TRRS, SW1 CherryMX, SW10 CherryMX, SW11 CherryMX, SW12 CherryMX, SW13 CherryMX, SW14 CherryMX, SW15 CherryMX, SW16 CherryMX, SW17 CherryMX, SW18 CherryMX, SW19 CherryMX, SW2 CherryMX, SW20 CherryMX, SW21 CherryMX, SW22 CherryMX, SW23 CherryMX, SW24 CherryMX, SW25 CherryMX, SW26 CherryMX, SW27 CherryMX, SW28 CherryMX, SW29 CherryMX, SW3 CherryMX, SW30 CherryMX, SW31 CherryMX, SW32 CherryMX, SW33 CherryMX, SW34 CherryMX, SW35 CherryMX, SW36 CherryMX, SW37 CherryMX, SW38 CherryMX, SW39 CherryMX, SW4 CherryMX, SW40 CherryMX, SW41 CherryMX, SW42 RotaryEncoder, SW43 CherryMX, SW44 CherryMX, SW45 CherryMX, SW46 CherryMX, SW47 CherryMX, SW48 CherryMX, SW49 CherryMX, SW5 CherryMX, SW50 CherryMX, SW51 CherryMX, SW52 CherryMX, SW53 RotaryEncoder, SW54 CherryMX, SW55 CherryMX, SW56 CherryMX, SW57 CherryMX, SW58 CherryMX, SW59 CherryMX, SW6 CherryMX, SW60 CherryMX, SW61 CherryMX, SW7 CherryMX, SW8 CherryMX, SW9 CherryMX, U1 Pico, U2 Pico

Commit message: Added branding to pcb
Other:
- board text added: "Split-Kola"
