File: ergo-kola/pcb/ergo-kola/ergo-kola.kicad_pcb (KiCad board)
At the start: 2 copper layers, 360.4 x 103.2 mm, 185 parts, among them J1 L_TRRS, J2 L_TRRS, SW1 CherryMX, SW10 CherryMX, SW11 CherryMX, SW12 CherryMX, SW13 CherryMX, SW14 CherryMX, SW15 CherryMX, SW16 CherryMX, SW17 CherryMX, SW18 CherryMX, SW19 CherryMX, SW2 CherryMX, SW20 CherryMX, SW21 CherryMX, SW22 CherryMX, SW23 CherryMX, SW24 CherryMX, SW25 CherryMX, SW26 CherryMX, SW27 CherryMX, SW28 CherryMX, SW29 CherryMX, SW3 CherryMX, SW30 CherryMX, SW31 CherryMX, SW32 CherryMX, SW33 CherryMX, SW34 CherryMX, SW35 CherryMX, SW36 CherryMX, SW37 CherryMX, SW38 CherryMX, SW39 CherryMX, SW4 CherryMX, SW40 CherryMX, SW41 CherryMX, SW42 RotaryEncoder, SW43 CherryMX, SW44 CherryMX, SW45 CherryMX, SW46 CherryMX, SW47 CherryMX, SW48 CherryMX, SW49 CherryMX, SW5 CherryMX, SW50 CherryMX, SW51 CherryMX, SW52 CherryMX, SW53 RotaryEncoder, SW54 CherryMX, SW55 CherryMX, SW56 CherryMX, SW57 CherryMX, SW58 CherryMX, SW59 CherryMX, SW6 CherryMX, SW60 CherryMX, SW61 CherryMX, SW7 CherryMX, SW8 CherryMX, SW9 CherryMX, U1 Pico, U2 Pico

Commit message: Autolayout did not work (experiment), manually doing it via spreadsheet
Parts:
- removed D1.5, D10.5, D11.5, D12.5, D13.5, D14.5, D15.5, D16.5, D17.5, D18.5, D19.5, D2.5, D20.5, D21.5, D22.5, D23.5, D24.5, D25.5, D26.5, D27.5, D28.5, D29.5, D3.5, D30.5, D31.5, D35.5, D36.5, D37.5, D38.5, D39.5, D4.5, D40.5, D41.5, D42.5, D43.5, D44.5, D45.5, D46.5, D47.5, D48.5, D49.5, D5.5, D50.5, D51.5, D52.5, D53.5, D54.5, D55.5, D56.5, D57.5, D58.5, D59.5, D6.5, D60.5, D61.5, D62.5, D63.5, D64.5, D7.5, D8.5, D9.5: WS2812B, footprints:SK6812-MINI-E
- removed D53, D54, D55, D56, D57, D58, D59: D, Diode_SMD:D_SOD-123
- removed SW53: RotaryEncoder, Rotary_Encoder:RotaryEncoder_Alps_EC12E_Vertical_H20mm
- removed SW54, SW61: CherryMX, CherryMX_PCB_KailhSocket_StabWireBottom:CherryMX_2.25u_PCB_KailhSocket_StabWireBottom
- removed SW55, SW60: CherryMX, CherryMX_PCB_KailhSocket:CherryMX_1.50u_PCB_KailhSocket
- removed SW56, SW59: CherryMX, CherryMX_PCB_KailhSocket:CherryMX_1.25u_PCB_KailhSocket
- removed SW57, SW58: CherryMX, CherryMX_PCB_KailhSocket_StabWireBottom:CherryMX_2.75u_PCB_KailhSocket_StabWireBottom
- added C1: C 100uf, Capacitor_SMD:C_0805_2012Metric_Pad1.18x1.45mm_HandSolder, F.Cu at (-4.23, -43.1)
- added C10: C 100uf, Capacitor_SMD:C_0805_2012Metric_Pad1.18x1.45mm_HandSolder, F.Cu at (-4.23, -16.0)
- added C11: C 100uf, Capacitor_SMD:C_0805_2012Metric_Pad1.18x1.45mm_HandSolder, F.Cu at (-4.23, -13.0)
- added C12: C 100uf, Capacitor_SMD:C_0805_2012Metric_Pad1.18x1.45mm_HandSolder, F.Cu at (0.58, -43.1)
- added C13: C 100uf, Capacitor_SMD:C_0805_2012Metric_Pad1.18x1.45mm_HandSolder, F.Cu at (0.58, -40.1)
- added C14: C 100uf, Capacitor_SMD:C_0805_2012Metric_Pad1.18x1.45mm_HandSolder, F.Cu at (0.58, -37.1)
- added C15: C 100uf, Capacitor_SMD:C_0805_2012Metric_Pad1.18x1.45mm_HandSolder, F.Cu at (0.58, -34.1)
- added C16: C 100uf, Capacitor_SMD:C_0805_2012Metric_Pad1.18x1.45mm_HandSolder, F.Cu at (0.58, -31.1)
- added C17: C 100uf, Capacitor_SMD:C_0805_2012Metric_Pad1.18x1.45mm_HandSolder, F.Cu at (0.58, -28.0)
- added C18: C 100uf, Capacitor_SMD:C_0805_2012Metric_Pad1.18x1.45mm_HandSolder, F.Cu at (0.58, -25.0)
- added C19: C 100uf, Capacitor_SMD:C_0805_2012Metric_Pad1.18x1.45mm_HandSolder, F.Cu at (0.58, -22.0)
- added C2: C 100uf, Capacitor_SMD:C_0805_2012Metric_Pad1.18x1.45mm_HandSolder, F.Cu at (-4.23, -40.1)
- added C20: C 100uf, Capacitor_SMD:C_0805_2012Metric_Pad1.18x1.45mm_HandSolder, F.Cu at (0.58, -19.0)
- added C21: C 100uf, Capacitor_SMD:C_0805_2012Metric_Pad1.18x1.45mm_HandSolder, F.Cu at (0.58, -16.0)
- added C23: C 100uf, Capacitor_SMD:C_0805_2012Metric_Pad1.18x1.45mm_HandSolder, F.Cu at (5.39, -43.1)
- added C24: C 100uf, Capacitor_SMD:C_0805_2012Metric_Pad1.18x1.45mm_HandSolder, F.Cu at (5.39, -40.1)
- added C25: C 100uf, Capacitor_SMD:C_0805_2012Metric_Pad1.18x1.45mm_HandSolder, F.Cu at (5.39, -37.1)
- added C26: C 100uf, Capacitor_SMD:C_0805_2012Metric_Pad1.18x1.45mm_HandSolder, F.Cu at (5.39, -34.1)
- added C27: C 100uf, Capacitor_SMD:C_0805_2012Metric_Pad1.18x1.45mm_HandSolder, F.Cu at (5.39, -31.1)
- added C28: C 100uf, Capacitor_SMD:C_0805_2012Metric_Pad1.18x1.45mm_HandSolder, F.Cu at (5.39, -28.0)
- added C29: C 100uf, Capacitor_SMD:C_0805_2012Metric_Pad1.18x1.45mm_HandSolder, F.Cu at (5.39, -25.0)
- added C3: C 100uf, Capacitor_SMD:C_0805_2012Metric_Pad1.18x1.45mm_HandSolder, F.Cu at (-4.23, -37.1)
- added C30: C 100uf, Capacitor_SMD:C_0805_2012Metric_Pad1.18x1.45mm_HandSolder, F.Cu at (5.39, -22.0)
- added C31: C 100uf, Capacitor_SMD:C_0805_2012Metric_Pad1.18x1.45mm_HandSolder, F.Cu at (5.39, -19.0)
- added C32: C 100uf, Capacitor_SMD:C_0805_2012Metric_Pad1.18x1.45mm_HandSolder, F.Cu at (5.39, -16.0)
- added C33: C 100uf, Capacitor_SMD:C_0805_2012Metric_Pad1.18x1.45mm_HandSolder, F.Cu at (5.39, -13.0)
- added C34: C 100uf, Capacitor_SMD:C_0805_2012Metric_Pad1.18x1.45mm_HandSolder, F.Cu at (10.2, -43.1)
- added C35: C 100uf, Capacitor_SMD:C_0805_2012Metric_Pad1.18x1.45mm_HandSolder, F.Cu at (10.2, -40.1)
- added C36: C 100uf, Capacitor_SMD:C_0805_2012Metric_Pad1.18x1.45mm_HandSolder, F.Cu at (10.2, -37.1)
- added C37: C 100uf, Capacitor_SMD:C_0805_2012Metric_Pad1.18x1.45mm_HandSolder, F.Cu at (10.2, -34.1)
- added C38: C 100uf, Capacitor_SMD:C_0805_2012Metric_Pad1.18x1.45mm_HandSolder, F.Cu at (10.2, -31.1)
- added C39: C 100uf, Capacitor_SMD:C_0805_2012Metric_Pad1.18x1.45mm_HandSolder, F.Cu at (10.2, -28.0)
- added C4: C 100uf, Capacitor_SMD:C_0805_2012Metric_Pad1.18x1.45mm_HandSolder, F.Cu at (-4.23, -34.1)
- added C40: C 100uf, Capacitor_SMD:C_0805_2012Metric_Pad1.18x1.45mm_HandSolder, F.Cu at (10.2, -25.0)
- added C41: C 100uf, Capacitor_SMD:C_0805_2012Metric_Pad1.18x1.45mm_HandSolder, F.Cu at (10.2, -22.0)
- added C42: C 100uf, Capacitor_SMD:C_0805_2012Metric_Pad1.18x1.45mm_HandSolder, F.Cu at (10.2, -19.0)
- added C43: C 100uf, Capacitor_SMD:C_0805_2012Metric_Pad1.18x1.45mm_HandSolder, F.Cu at (10.2, -16.0)
- added C45: C 100uf, Capacitor_SMD:C_0805_2012Metric_Pad1.18x1.45mm_HandSolder, F.Cu at (15.0, -43.1)
- added C46: C 100uf, Capacitor_SMD:C_0805_2012Metric_Pad1.18x1.45mm_HandSolder, F.Cu at (15.0, -40.1)
- added C47: C 100uf, Capacitor_SMD:C_0805_2012Metric_Pad1.18x1.45mm_HandSolder, F.Cu at (15.0, -37.1)
- added C48: C 100uf, Capacitor_SMD:C_0805_2012Metric_Pad1.18x1.45mm_HandSolder, F.Cu at (15.0, -34.1)
- added C49: C 100uf, Capacitor_SMD:C_0805_2012Metric_Pad1.18x1.45mm_HandSolder, F.Cu at (15.0, -31.1)
- added C5: C 100uf, Capacitor_SMD:C_0805_2012Metric_Pad1.18x1.45mm_HandSolder, F.Cu at (-4.23, -31.1)
- added C50: C 100uf, Capacitor_SMD:C_0805_2012Metric_Pad1.18x1.45mm_HandSolder, F.Cu at (15.0, -28.0)
- added C51: C 100uf, Capacitor_SMD:C_0805_2012Metric_Pad1.18x1.45mm_HandSolder, F.Cu at (15.0, -25.0)
- added C52: C 100uf, Capacitor_SMD:C_0805_2012Metric_Pad1.18x1.45mm_HandSolder, F.Cu at (15.0, -22.0)
- added C53: C 100uf, Capacitor_SMD:C_0805_2012Metric_Pad1.18x1.45mm_HandSolder, F.Cu at (15.0, -19.0)
- added C54: C 100uf, Capacitor_SMD:C_0805_2012Metric_Pad1.18x1.45mm_HandSolder, F.Cu at (15.0, -16.0)
- added C55: C 100uf, Capacitor_SMD:C_0805_2012Metric_Pad1.18x1.45mm_HandSolder, F.Cu at (15.0, -13.0)
- added C6: C 100uf, Capacitor_SMD:C_0805_2012Metric_Pad1.18x1.45mm_HandSolder, F.Cu at (-4.23, -28.0)
- added C7: C 100uf, Capacitor_SMD:C_0805_2012Metric_Pad1.18x1.45mm_HandSolder, F.Cu at (-4.23, -25.0)
- added C8: C 100uf, Capacitor_SMD:C_0805_2012Metric_Pad1.18x1.45mm_HandSolder, F.Cu at (-4.23, -22.0)
- added C9: C 100uf, Capacitor_SMD:C_0805_2012Metric_Pad1.18x1.45mm_HandSolder, F.Cu at (-4.23, -19.0)
- added L1: WS2812B, footprints:SK6812-MINI-E, F.Cu at (-68.4, 11.6)
- added L10: WS2812B, footprints:SK6812-MINI-E, F.Cu at (-60.6, 11.6)
- added L11: WS2812B, footprints:SK6812-MINI-E, F.Cu at (-60.6, 16.4)
- added L12: WS2812B, footprints:SK6812-MINI-E, F.Cu at (-60.6, 21.3)
- added L13: WS2812B, footprints:SK6812-MINI-E, F.Cu at (-60.6, 26.2)
- added L14: WS2812B, footprints:SK6812-MINI-E, F.Cu at (-60.6, 31.1)
- added L15: WS2812B, footprints:SK6812-MINI-E, F.Cu at (-60.6, 36.0)
- added L16: WS2812B, footprints:SK6812-MINI-E, F.Cu at (-60.6, 40.9)
- added L17: WS2812B, footprints:SK6812-MINI-E, F.Cu at (-60.6, 45.8)
- added L18: WS2812B, footprints:SK6812-MINI-E, F.Cu at (-60.6, 50.7)
- added L19: WS2812B, footprints:SK6812-MINI-E, F.Cu at (-52.8, 11.6)
- added L2: WS2812B, footprints:SK6812-MINI-E, F.Cu at (-68.4, 16.4)
- added L20: WS2812B, footprints:SK6812-MINI-E, F.Cu at (-52.8, 16.4)
- added L21: WS2812B, footprints:SK6812-MINI-E, F.Cu at (-52.8, 21.3)
- added L22: WS2812B, footprints:SK6812-MINI-E, F.Cu at (-52.8, 26.2)
- added L23: WS2812B, footprints:SK6812-MINI-E, F.Cu at (-52.8, 31.1)
- added L24: WS2812B, footprints:SK6812-MINI-E, F.Cu at (-52.8, 36.0)
- added L25: WS2812B, footprints:SK6812-MINI-E, F.Cu at (-52.8, 40.9)
- added L26: WS2812B, footprints:SK6812-MINI-E, F.Cu at (-52.8, 45.8)
- added L27: WS2812B, footprints:SK6812-MINI-E, F.Cu at (-52.8, 50.7)
- added L28: WS2812B, footprints:SK6812-MINI-E, F.Cu at (-45.0, 11.6)
- added L29: WS2812B, footprints:SK6812-MINI-E, F.Cu at (-45.0, 16.4)
- added L3: WS2812B, footprints:SK6812-MINI-E, F.Cu at (-68.4, 21.3)
- added L30: WS2812B, footprints:SK6812-MINI-E, F.Cu at (-45.0, 21.3)
- added L31: WS2812B, footprints:SK6812-MINI-E, F.Cu at (-45.0, 26.2)
- added L32: WS2812B, footprints:SK6812-MINI-E, F.Cu at (-45.0, 31.1)
- added L33: WS2812B, footprints:SK6812-MINI-E, F.Cu at (-45.0, 36.0)
- added L34: WS2812B, footprints:SK6812-MINI-E, F.Cu at (-45.0, 40.9)
- added L35: WS2812B, footprints:SK6812-MINI-E, F.Cu at (-45.0, 45.8)
- added L36: WS2812B, footprints:SK6812-MINI-E, F.Cu at (-45.0, 50.7)
- added L37: WS2812B, footprints:SK6812-MINI-E, F.Cu at (-37.2, 11.6)
- added L38: WS2812B, footprints:SK6812-MINI-E, F.Cu at (-37.2, 16.4)
- added L39: WS2812B, footprints:SK6812-MINI-E, F.Cu at (-37.2, 21.3)
- added L4: WS2812B, footprints:SK6812-MINI-E, F.Cu at (-68.4, 26.2)
- added L40: WS2812B, footprints:SK6812-MINI-E, F.Cu at (-37.2, 26.2)
- added L41: WS2812B, footprints:SK6812-MINI-E, F.Cu at (-37.2, 31.1)
- added L42: WS2812B, footprints:SK6812-MINI-E, F.Cu at (-37.2, 36.0)
- added L43: WS2812B, footprints:SK6812-MINI-E, F.Cu at (-37.2, 40.9)
- added L44: WS2812B, footprints:SK6812-MINI-E, F.Cu at (-37.2, 45.8)
- added L45: WS2812B, footprints:SK6812-MINI-E, F.Cu at (-37.2, 50.7)
- added L46: WS2812B, footprints:SK6812-MINI-E, F.Cu at (-29.4, 11.6)
- added L47: WS2812B, footprints:SK6812-MINI-E, F.Cu at (-29.4, 16.4)
- added L48: WS2812B, footprints:SK6812-MINI-E, F.Cu at (-29.4, 21.3)
- added L49: WS2812B, footprints:SK6812-MINI-E, F.Cu at (-29.4, 26.2)
- added L5: WS2812B, footprints:SK6812-MINI-E, F.Cu at (-68.4, 31.1)
- added L50: WS2812B, footprints:SK6812-MINI-E, F.Cu at (-29.4, 31.1)
- added L51: WS2812B, footprints:SK6812-MINI-E, F.Cu at (-29.4, 36.0)
- added L52: WS2812B, footprints:SK6812-MINI-E, F.Cu at (-29.4, 40.9)
- added L6: WS2812B, footprints:SK6812-MINI-E, F.Cu at (-68.4, 36.0)
- added L7: WS2812B, footprints:SK6812-MINI-E, F.Cu at (-68.4, 40.9)
- added L8: WS2812B, footprints:SK6812-MINI-E, F.Cu at (-68.4, 45.8)
- added L9: WS2812B, footprints:SK6812-MINI-E, F.Cu at (-68.4, 50.7)
- SW13: footprint CherryMX_PCB_KailhSocket_StabWireBottom:CherryMX_2.00u_PCB_KailhSocket_StabWireBottom -> CherryMX_PCB_KailhSocket:CherryMX_1.00u_PCB_KailhSocket
- SW42: value RotaryEncoder -> CherryMX; footprint Rotary_Encoder:RotaryEncoder_Alps_EC12E_Vertical_H20mm -> CherryMX_PCB_KailhSocket:CherryMX_1.00u_PCB_KailhSocket
- moved SW41 318.3 mm to (61.5, 97.4), turned to -18 degrees
- moved SW25 291.4 mm to (47.3, 74.9), turned to -15 degrees
- moved U2 284.7 mm to (-36.2, -18.0), turned to 0 degrees
- moved D41 283.9 mm to (65.4, 101.9), turned to 72 degrees
- moved D49 272.5 mm to (101.5, 134.7), turned to 72 degrees
- moved J2 272.1 mm to (-21.0, -15.9), turned to 0 degrees
- moved SW27 267.2 mm to (109.9, 78.8), turned to -22 degrees
- moved SW13 264.3 mm to (98.3, 56.8), turned to -22 degrees
- moved U1 262.8 mm to (-60.3, -18.0), turned to 0 degrees
- moved SW11 262.8 mm to (52.2, 56.5), turned to -15 degrees
- moved SW37 261.1 mm to (42.4, 93.3), turned to -15 degrees
- moved D35 260.1 mm to (87.6, 96.8), turned to 68 degrees
- moved J1 248.9 mm to (-21.0, -23.6), turned to 0 degrees
- moved SW42 239.8 mm to (301.6, 97.4), turned to 18 degrees
- moved SW39 239.0 mm to (102.8, 96.4), turned to -22 degrees
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Connections:
- D13 pad 1: L_R1 -> L_R2
- D14 pad 1: L_R1 -> L_R2
- D19 pad 1: L_R2 -> L_R3
- D20 pad 1: L_R2 -> L_R3
- D21 pad 1: L_R2 -> L_R3
- D25 pad 1: L_R3 -> L_R4
- D26 pad 1: L_R3 -> L_R4
- D27 pad 1: L_R4 -> R_R0
- D28 pad 1: L_R4 -> R_R0
- D29 pad 1: L_R4 -> R_R0
- D30 pad 1: L_R4 -> R_R0
- D33 pad 1: R_R0 -> R_R1
- D34 pad 1: R_R0 -> R_R1
- D35 pad 1: R_R0 -> R_R1
- D36 pad 1: R_R0 -> R_R1
- D39 pad 1: R_R1 -> R_R2
- D40 pad 1: R_R1 -> R_R2
- D41 pad 1: R_R1 -> R_R2
- D42 pad 1: R_R1 -> R_R2
- D43 pad 1: R_R1 -> R_R2
- D45 pad 1: R_R2 -> R_R3
- D46 pad 1: R_R2 -> R_R3
- D47 pad 1: R_R2 -> R_R3
- D48 pad 1: R_R2 -> R_R3
- D49 pad 1: R_R2 -> R_R3
- D50 pad 1: R_R2 -> R_R3
- D51 pad 1: R_R3 -> R_R4
- D52 pad 1: R_R3 -> R_R4
- D7 pad 1: L_R0 -> L_R1
- J1 pad 3: L_GP1 -> L_RX
- J1 pad 4: L_GP0 -> L_TX
- J2 pad 3: R_GP1 -> L_TX
- J2 pad 4: R_GP0 -> R_RX
- SW10 pad 1: R_C9 -> L_C3
- SW10 pad 2: Net-(D33-A) -> Net-(D10-A)
- SW11 pad 1: R_C10 -> L_C4
- SW11 pad 2: Net-(D34-A) -> Net-(D11-A)
- SW12 pad 1: R_C11 -> L_C5
- SW12 pad 2: Net-(D35-A) -> Net-(D12-A)
- SW13 pad 1: R_C12 -> L_C0
- SW13 pad 2: Net-(D36-A) -> Net-(D13-A)
- SW14 pad 1: L_C0 -> L_C1
- SW14 pad 2: Net-(D8-A) -> Net-(D14-A)
- SW15 pad 1: L_C1 -> L_C2
- SW15 pad 2: Net-(D9-A) -> Net-(D15-A)
- SW16 pad 1: L_C2 -> L_C3
- SW16 pad 2: Net-(D10-A) -> Net-(D16-A)
- SW17 pad 1: L_C3 -> L_C4
- SW17 pad 2: Net-(D11-A) -> Net-(D17-A)
- SW18 pad 1: L_C4 -> L_C5
- SW18 pad 2: Net-(D12-A) -> Net-(D18-A)
- SW19 pad 1: L_C5 -> L_C0
- SW19 pad 2: Net-(D13-A) -> Net-(D19-A)
- SW20 pad 1: L_C6 -> L_C1
- SW20 pad 2: Net-(D14-A) -> Net-(D20-A)
- SW21 pad 1: R_C7 -> L_C2
- SW21 pad 2: Net-(D37-A) -> Net-(D21-A)
- SW22 pad 1: R_C8 -> L_C3
- SW22 pad 2: Net-(D38-A) -> Net-(D22-A)
- SW23 pad 1: R_C9 -> L_C4
- SW23 pad 2: Net-(D39-A) -> Net-(D23-A)
- SW24 pad 1: R_C10 -> L_C5
- SW24 pad 2: Net-(D40-A) -> Net-(D24-A)
- SW25 pad 1: R_C11 -> L_C4
- SW25 pad 2: Net-(D41-A) -> Net-(D25-A)
- SW26 pad 1: R_C12 -> L_C5
- SW26 pad 2: Net-(D42-A) -> Net-(D26-A)
- SW27 pad 1: R_C13 -> R_C6
- SW27 pad 2: Net-(D43-A) -> Net-(D27-A)
- SW28 pad 1: L_C0 -> R_C7
- SW28 pad 2: Net-(D15-A) -> Net-(D28-A)
- SW29 pad 1: L_C1 -> R_C8
- SW29 pad 2: Net-(D16-A) -> Net-(D29-A)
- SW30 pad 1: L_C2 -> R_C9
- SW30 pad 2: Net-(D17-A) -> Net-(D30-A)
- SW31 pad 1: L_C3 -> R_C10
- SW31 pad 2: Net-(D18-A) -> Net-(D31-A)
- SW32 pad 1: L_C4 -> R_C11
- SW32 pad 2: Net-(D19-A) -> Net-(D32-A)
- SW33 pad 1: L_C5 -> R_C6
- SW33 pad 2: Net-(D20-A) -> Net-(D33-A)
- SW34 pad 1: L_C6 -> R_C7
- SW34 pad 2: Net-(D21-A) -> Net-(D34-A)
- SW35 pad 1: R_C7 -> R_C8
- SW35 pad 2: Net-(D44-A) -> Net-(D35-A)
- SW36 pad 1: R_C8 -> R_C9
- SW36 pad 2: Net-(D45-A) -> Net-(D36-A)
- SW37 pad 1: R_C9 -> R_C10
- SW37 pad 2: Net-(D46-A) -> Net-(D37-A)
- SW38 pad 1: R_C10 -> R_C11
- SW38 pad 2: Net-(D47-A) -> Net-(D38-A)
- SW39 pad 1: R_C11 -> R_C6
- SW39 pad 2: Net-(D48-A) -> Net-(D39-A)
- SW40 pad 1: R_C12 -> R_C7
- SW40 pad 2: Net-(D49-A) -> Net-(D40-A)
- SW41 pad 1: R_C13 -> R_C8
- SW41 pad 2: Net-(D50-A) -> Net-(D41-A)
- SW43 pad 1: L_C2 -> R_C10
- SW43 pad 2: Net-(D22-A) -> Net-(D43-A)
- SW44 pad 1: L_C3 -> R_C11
- SW44 pad 2: Net-(D23-A) -> Net-(D44-A)
- SW45 pad 1: L_C4 -> R_C6
- SW45 pad 2: Net-(D24-A) -> Net-(D45-A)
- SW46 pad 1: L_C5 -> R_C7
- SW46 pad 2: Net-(D25-A) -> Net-(D46-A)
- SW47 pad 1: L_C6 -> R_C8
- SW47 pad 2: Net-(D26-A) -> Net-(D47-A)
- SW48 pad 1: R_C7 -> R_C9
- SW48 pad 2: Net-(D51-A) -> Net-(D48-A)
- SW49 pad 1: R_C8 -> R_C10
- SW49 pad 2: Net-(D52-A) -> Net-(D49-A)
- SW50 pad 1: R_C9 -> R_C11
- SW50 pad 2: Net-(D53-A) -> Net-(D50-A)
- SW51 pad 1: R_C10 -> R_C6
- SW51 pad 2: Net-(D54-A) -> Net-(D51-A)
- SW52 pad 1: R_C11 -> R_C7
- SW52 pad 2: Net-(D55-A) -> Net-(D52-A)
- SW7 pad 1: L_C6 -> L_C0
- SW8 pad 1: R_C7 -> L_C1
- SW8 pad 2: Net-(D31-A) -> Net-(D8-A)
- SW9 pad 1: R_C8 -> L_C2
- SW9 pad 2: Net-(D32-A) -> Net-(D9-A)
- U1 pad 1: L_GP0 -> L_RGB
- U1 pad 17: L_C6 -> unconnected-(U1-GPIO13-Pad17)_1
- U1 pad 2: L_GP1 -> unconnected-(U1-GPIO1-Pad2)_1
- U1 pad 20: L_RGB -> unconnected-(U1-GPIO15-Pad20)_1
- U1 pad 22: unconnected-(U1-GPIO17-Pad22)_1 -> L_R0
- U1 pad 24: unconnected-(U1-GPIO18-Pad24) -> L_R1
- U1 pad 25: unconnected-(U1-GPIO19-Pad25)_1 -> L_R2
- U1 pad 26: L_ECB -> L_R3
- U1 pad 27: L_ECA -> L_R4
- U1 pad 4: L_R0 -> unconnected-(U1-GPIO2-Pad4)_1
- U1 pad 5: L_R1 -> unconnected-(U1-GPIO3-Pad5)
- U1 pad 6: L_R2 -> L_TX
- U1 pad 7: L_R3 -> L_RX
- U1 pad 9: L_R4 -> unconnected-(U1-GPIO6-Pad9)_1
- U2 pad 1: R_GP0 -> R_RGB
- U2 pad 17: R_C13 -> unconnected-(U2-GPIO13-Pad17)
- U2 pad 2: R_GP1 -> unconnected-(U2-GPIO1-Pad2)_1
- U2 pad 20: R_RGB -> unconnected-(U2-GPIO15-Pad20)
- U2 pad 22: unconnected-(U2-GPIO17-Pad22)_1 -> R_R0
- U2 pad 24: unconnected-(U2-GPIO18-Pad24) -> R_R1
- U2 pad 25: unconnected-(U2-GPIO19-Pad25) -> R_R2
- U2 pad 26: R_ECB -> R_R3
- U2 pad 27: R_ECA -> R_R4
- U2 pad 4: R_R0 -> unconnected-(U2-GPIO2-Pad4)
- U2 pad 5: R_R1 -> unconnected-(U2-GPIO3-Pad5)
- U2 pad 6: R_R2 -> R_TX
- U2 pad 7: R_R3 -> R_RX
- U2 pad 9: R_R4 -> unconnected-(U2-GPIO6-Pad9)
Routing:
- net L_VBUS: track 797.7 -> 0.00 mm, vias 8 -> 0
- net R_VBUS: track 787.5 -> 0.00 mm, vias 8 -> 0
- net R_C11: track 278.5 -> 0.00 mm, vias 5 -> 0
- net R_C12: track 261.3 -> 0.00 mm, vias 3 -> 0
- net L_C2: track 258.4 -> 0.00 mm, vias 6 -> 0
- net R_C13: track 234.4 -> 0.00 mm, vias 2 -> 0
- net R_C10: track 230.4 -> 0.00 mm, vias 5 -> 0
- net R_ECB: track 227.2 -> 0.00 mm, vias 3 -> 0
- net L_C0: track 218.7 -> 0.00 mm, vias 4 -> 0
- net L_C3: track 215.1 -> 0.00 mm, vias 6 -> 0
- net R_R4: track 213.0 -> 0.00 mm
- net R_ECA: track 210.3 -> 0.00 mm, vias 2 -> 0
- net L_C4: track 208.0 -> 0.00 mm, vias 6 -> 0
- net L_C1: track 207.7 -> 0.00 mm, vias 4 -> 0
- net R_C9: track 199.2 -> 0.00 mm, vias 5 -> 0
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- removed copper zone on B.Cu, net GND
- removed copper zone on F.Cu, net GND
Other:
- board text removed: "Split-Kola"
