File: ergo-kola/pcb/ergo-kola/ergo-kola.kicad_pcb (KiCad board)
At the start: 2 copper layers, 341.1 x 127.2 mm, 212 parts, among them J1 L_TRRS, J2 L_TRRS, SW1 CherryMX, SW10 CherryMX, SW11 CherryMX, SW12 CherryMX, SW13 CherryMX, SW14 CherryMX, SW15 CherryMX, SW16 CherryMX, SW17 CherryMX, SW18 CherryMX, SW19 CherryMX, SW2 CherryMX, SW20 CherryMX, SW21 CherryMX, SW22 CherryMX, SW23 CherryMX, SW24 CherryMX, SW25 CherryMX, SW26 CherryMX, SW27 CherryMX, SW28 CherryMX, SW29 CherryMX, SW3 CherryMX, SW30 CherryMX, SW31 CherryMX, SW32 CherryMX, SW33 CherryMX, SW34 CherryMX, SW35 CherryMX, SW36 CherryMX, SW37 CherryMX, SW38 CherryMX, SW39 CherryMX, SW4 CherryMX, SW40 CherryMX, SW41 CherryMX, SW42 CherryMX, SW43 CherryMX, SW44 CherryMX, SW45 CherryMX, SW46 CherryMX, SW47 CherryMX, SW48 CherryMX, SW49 CherryMX, SW5 CherryMX, SW50 CherryMX, SW51 CherryMX, SW52 CherryMX, SW6 CherryMX, SW7 CherryMX, SW8 CherryMX, SW9 CherryMX, U1 Pico, U2 Pico

Commit message: Finished PCB and Case!
Routing:
- net (no net): vias 0 -> 1

Commit message: Neopixels power fixed
Parts:
- removed C19, C20, C21, C22, C23, C24, C25, C26, C27, C28, C29, C30, C31, C32, C33, C34, C35, C36, C37, C38, C39, C40, C41, C42, C43, C44, C45, C46, C47, C48, C49, C50, C51, C52: C 100uf, Capacitor_SMD:C_0805_2012Metric_Pad1.18x1.45mm_HandSolder
- C1, C10, C11, C12, C13, C14, C15, C16, C17, C18, C2, C3, C4, C5, C6, C7, C8, C9: value C 100uf -> C 10uf
- moved C2 292.5 mm to (51.8, 47.4), turned to 90 degrees
- moved C6 282.7 mm to (42.0, 84.8), turned to 90 degrees
- moved C4 251.0 mm to (46.7, 66.1), turned to 90 degrees
- moved C8 247.9 mm to (35.3, 100.6), turned to 90 degrees
- moved C17 206.9 mm to (269.0, 128.4), turned to 20 degrees
- moved C11 193.4 mm to (243.2, 74.7), turned to 0 degrees
- moved C13 159.7 mm to (252.2, 93.6), turned to 0 degrees
- moved C15 150.3 mm to (258.1, 111.5), turned to 0 degrees
- moved C12 101.8 mm to (251.0, 91.1), turned to 0 degrees
- moved C7 100.0 mm to (32.9, 98.6), turned to 70 degrees
- moved C18 87.6 mm to (284.4, 144.9), turned to 90 degrees
- moved C9 85.9 mm to (94.2, 135.5), turned to 110 degrees
- moved C14 65.0 mm to (256.3, 108.6), turned to 0 degrees
- moved C3 61.5 mm to (43.9, 66.5), turned to 90 degrees
- moved C16 60.4 mm to (267.7, 126.7), turned to 20 degrees
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Connections:
- C1 pad 1: L_VBUS -> GND
- C1 pad 2: Net-(L1-VDD) -> L_VBUS
- C10 pad 1: Net-(L20-VDD) -> GND
- C10 pad 2: Net-(L10-VDD) -> R_VBUS
- C11 pad 1: L_VBUS -> GND
- C11 pad 2: Net-(L11-VDD) -> R_VBUS
- C12 pad 1: Net-(L18-VDD) -> GND
- C12 pad 2: Net-(L12-VDD) -> R_VBUS
- C13 pad 1: Net-(L17-VDD) -> GND
- C13 pad 2: Net-(L13-VDD) -> R_VBUS
- C14 pad 1: Net-(L16-VDD) -> GND
- C14 pad 2: Net-(L14-VDD) -> R_VBUS
- C15 pad 1: Net-(L13-VDD) -> GND
- C15 pad 2: Net-(L15-VDD) -> R_VBUS
- C16 pad 1: Net-(L22-VDD) -> GND
- C16 pad 2: Net-(L16-VDD) -> R_VBUS
- C17 pad 1: Net-(L11-VDD) -> GND
- C17 pad 2: Net-(L17-VDD) -> R_VBUS
- C18 pad 1: Net-(L14-VDD) -> GND
- C18 pad 2: Net-(L18-VDD) -> R_VBUS
- C2 pad 1: Net-(L6-VDD) -> GND
- C2 pad 2: Net-(L2-VDD) -> L_VBUS
- C3 pad 1: Net-(L5-VDD) -> GND
- C3 pad 2: Net-(L3-VDD) -> L_VBUS
- C4 pad 1: Net-(L8-VDD) -> GND
- C4 pad 2: Net-(L4-VDD) -> L_VBUS
- C5 pad 1: Net-(L1-VDD) -> GND
- C5 pad 2: Net-(L5-VDD) -> L_VBUS
- C6 pad 1: Net-(L4-VDD) -> GND
- C6 pad 2: Net-(L6-VDD) -> L_VBUS
- C7 pad 1: Net-(L3-VDD) -> GND
- C7 pad 2: Net-(L7-VDD) -> L_VBUS
- C8 pad 1: Net-(L10-VDD) -> GND
- C8 pad 2: Net-(L8-VDD) -> L_VBUS
- C9 pad 1: Net-(L7-VDD) -> GND
- C9 pad 2: Net-(L9-VDD) -> L_VBUS
- L1 pad 1: Net-(L1-VDD) -> L_VBUS
- L10 pad 1: Net-(L10-VDD) -> R_VBUS
- L11 pad 1: Net-(L11-VDD) -> L_VBUS
- L12 pad 1: Net-(L12-VDD) -> R_VBUS
- L13 pad 1: Net-(L13-VDD) -> L_VBUS
- L14 pad 1: Net-(L14-VDD) -> R_VBUS
- L15 pad 1: Net-(L15-VDD) -> L_VBUS
- L16 pad 1: Net-(L16-VDD) -> R_VBUS
- L17 pad 1: Net-(L17-VDD) -> L_VBUS
- L18 pad 1: Net-(L18-VDD) -> R_VBUS
- L19 pad 1: Net-(L19-VDD) -> L_VBUS
- L2 pad 1: Net-(L2-VDD) -> R_VBUS
- L20 pad 1: Net-(L20-VDD) -> R_VBUS
- L21 pad 1: Net-(L21-VDD) -> L_VBUS
- L22 pad 1: Net-(L22-VDD) -> R_VBUS
- L23 pad 1: Net-(L23-VDD) -> L_VBUS
- L24 pad 1: Net-(L24-VDD) -> R_VBUS
- L25 pad 1: Net-(L25-VDD) -> L_VBUS
- L26 pad 1: Net-(L26-VDD) -> R_VBUS
- L27 pad 1: Net-(L27-VDD) -> L_VBUS
- L28 pad 1: Net-(L28-VDD) -> R_VBUS
- L29 pad 1: Net-(L29-VDD) -> L_VBUS
- L3 pad 1: Net-(L3-VDD) -> L_VBUS
- L30 pad 1: Net-(L30-VDD) -> R_VBUS
- L31 pad 1: Net-(L31-VDD) -> L_VBUS
- L32 pad 1: Net-(L32-VDD) -> R_VBUS
- L33 pad 1: Net-(L33-VDD) -> L_VBUS
- L34 pad 1: Net-(L34-VDD) -> R_VBUS
- L35 pad 1: Net-(L35-VDD) -> L_VBUS
- L36 pad 1: Net-(L36-VDD) -> R_VBUS
- L37 pad 1: Net-(L37-VDD) -> L_VBUS
- L38 pad 1: Net-(L38-VDD) -> R_VBUS
- L39 pad 1: Net-(L39-VDD) -> L_VBUS
- L4 pad 1: Net-(L4-VDD) -> R_VBUS
- L40 pad 1: Net-(L40-VDD) -> R_VBUS
- L41 pad 1: Net-(L41-VDD) -> L_VBUS
- L42 pad 1: Net-(L42-VDD) -> R_VBUS
- L43 pad 1: Net-(L43-VDD) -> L_VBUS
- L44 pad 1: Net-(L44-VDD) -> R_VBUS
- L45 pad 1: Net-(L45-VDD) -> L_VBUS
- L46 pad 1: Net-(L46-VDD) -> R_VBUS
- L47 pad 1: Net-(L47-VDD) -> L_VBUS
- L48 pad 1: Net-(L48-VDD) -> R_VBUS
- L49 pad 1: Net-(L49-VDD) -> L_VBUS
- L5 pad 1: Net-(L5-VDD) -> L_VBUS
- L50 pad 1: Net-(L50-VDD) -> R_VBUS
- L51 pad 1: Net-(L51-VDD) -> L_VBUS
- L52 pad 1: Net-(L52-VDD) -> R_VBUS
- L6 pad 1: Net-(L6-VDD) -> R_VBUS
- L7 pad 1: Net-(L7-VDD) -> L_VBUS
- L8 pad 1: Net-(L8-VDD) -> R_VBUS
- L9 pad 1: Net-(L9-VDD) -> L_VBUS
- U2 pad 16: R_C12 -> unconnected-(U2-GPIO12-Pad16)
Routing:
- net R_VBUS: track 169.3 -> 675.1 mm, vias 4 -> 36
- net L_VBUS: track 317.2 -> 815.8 mm, vias 5 -> 44
- net Net-(L5-VDD): track 27.8 -> 0.00 mm, vias 2 -> 0
- net Net-(L4-VDD): track 27.7 -> 0.00 mm, vias 2 -> 0
- net Net-(L14-VDD): track 26.7 -> 0.00 mm, vias 2 -> 0
- net Net-(L36-VDD): track 25.9 -> 0.00 mm
- net Net-(L17-VDD): track 25.8 -> 0.00 mm, vias 2 -> 0
- net Net-(L24-VDD): track 25.7 -> 0.00 mm, vias 2 -> 0
- net Net-(L29-VDD): track 25.1 -> 0.00 mm, vias 2 -> 0
- net Net-(L41-VDD): track 23.1 -> 0.00 mm
- net Net-(L6-VDD): track 22.1 -> 0.00 mm, vias 2 -> 0
- net Net-(L1-VDD): track 21.6 -> 0.00 mm, vias 2 -> 0
- net Net-(L49-VDD): track 21.3 -> 0.00 mm
- net Net-(L18-VDD): track 21.1 -> 0.00 mm, vias 2 -> 0
- net Net-(L11-VDD): track 20.6 -> 0.00 mm, vias 2 -> 0
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