File: ergo-kola/pcb/ergo-kola/ergo-kola.kicad_sch (KiCad schematic)
At the start: 166 parts, among them J1 L_TRRS, J2 L_TRRS, SW1 CherryMX, SW10 CherryMX, SW11 CherryMX, SW12 CherryMX, SW13 CherryMX, SW14 CherryMX, SW15 CherryMX, SW16 CherryMX, SW17 CherryMX, SW18 CherryMX, SW19 CherryMX, SW2 CherryMX, SW20 CherryMX, SW21 CherryMX, SW22 CherryMX, SW23 CherryMX, SW24 CherryMX, SW25 CherryMX, SW26 CherryMX, SW27 CherryMX, SW28 CherryMX, SW29 CherryMX, SW3 CherryMX, SW30 CherryMX, SW31 CherryMX, SW32 CherryMX, SW33 CherryMX, SW34 CherryMX, SW35 CherryMX, SW36 CherryMX, SW37 CherryMX, SW38 CherryMX, SW39 CherryMX, SW4 CherryMX, SW40 CherryMX, SW43 CherryMX, SW44 CherryMX, SW45 CherryMX, SW46 CherryMX, SW48 CherryMX, SW49 CherryMX, SW5 CherryMX, SW50 CherryMX, SW51 CherryMX, SW52 CherryMX, SW55 CherryMX, SW56 CherryMX, SW57 CherryMX, SW58 CherryMX, SW59 CherryMX, SW6 CherryMX, SW7 CherryMX, SW8 CherryMX, SW9 CherryMX, U1 Pico, U2 Pico

Commit message: Autolayout did not work (experiment), manually doing it via spreadsheet
Parts:
- removed D28, D57: D, Diode_SMD:D_SOD-123, symbol Device:D
- removed D30.5, D64.5: WS2812B, footprints:SK6812-MINI-E, symbol LED:WS2812B
- removed SW55: CherryMX, CherryMX_PCB_KailhSocket:CherryMX_1.50u_PCB_KailhSocket, symbol CherryMX:CherryMX
- removed SW59: CherryMX, CherryMX_PCB_KailhSocket:CherryMX_1.25u_PCB_KailhSocket, symbol CherryMX:CherryMX
- added C1, C10, C11, C12, C13, C14, C15, C16, C17, C18, C19, C2, C20, C21, C23, C24, C25, C26, C27, C28, C29, C3, C30, C31, C32, C33, C34, C35, C36, C37, C38, C39, C4, C40, C41, C42, C43, C45, C46, C47, C48, C49, C5, C50, C51, C52, C53, C54, C55, C6, C7, C8, C9: C 100uf, Capacitor_SMD:C_0805_2012Metric_Pad1.18x1.45mm_HandSolder, symbol Device:C
- SW25: renamed from SW56; footprint CherryMX_PCB_KailhSocket:CherryMX_1.25u_PCB_KailhSocket -> CherryMX_PCB_KailhSocket:CherryMX_1.00u_PCB_KailhSocket
- SW26: renamed from SW57; footprint CherryMX_PCB_KailhSocket_StabWireBottom:CherryMX_2.75u_PCB_KailhSocket_StabWireBottom -> CherryMX_PCB_KailhSocket:CherryMX_1.00u_PCB_KailhSocket
- SW32: renamed from SW13; footprint CherryMX_PCB_KailhSocket_StabWireBottom:CherryMX_2.00u_PCB_KailhSocket_StabWireBottom -> CherryMX_PCB_KailhSocket:CherryMX_1.00u_PCB_KailhSocket
- SW51: renamed from SW34; footprint CherryMX_PCB_KailhSocket_StabWireBottom:CherryMX_2.75u_PCB_KailhSocket_StabWireBottom -> CherryMX_PCB_KailhSocket:CherryMX_1.00u_PCB_KailhSocket
- SW52: renamed from SW58; footprint CherryMX_PCB_KailhSocket_StabWireBottom:CherryMX_2.75u_PCB_KailhSocket_StabWireBottom -> CherryMX_PCB_KailhSocket:CherryMX_1.00u_PCB_KailhSocket
- U1, U2: footprint RPi_Pico:RPi_Pico_SMD_TH -> MCU_RaspberryPi_and_Boards:RPi_Pico_SMD_TH
- renumbered D11 to D10, D12 to D11, D13 to D12, D15 to D13, D16 to D14, D17 to D15, D18 to D16, D19 to D17, D20 to D18, D7 to D19, D14 to D20, D22 to D21, D23 to D22, D24 to D23, D25 to D24, D29 to D25, D30 to D26, D31 to D27, D32 to D28, D33 to D29, D34 to D30, D35 to D31, D36 to D32, D37 to D33, D38 to D34, D39 to D35, D40 to D36, D41 to D37, D42 to D38, D44 to D39, D45 to D40, D46 to D41, D47 to D42, D48 to D43, D49 to D44, D51 to D45, D52 to D46, D53 to D47, D54 to D48, D55 to D49, D21 to D50, D26 to D51, D56 to D52, D8 to D7, D9 to D8, D10 to D9, D1.5 to L1, D11.5 to L10, D12.5 to L11, D13.5 to L12, D15.5 to L13, D16.5 to L14, D17.5 to L15, D18.5 to L16, D19.5 to L17, D20.5 to L18, D22.5 to L19, D2.5 to L2, D23.5 to L20, D24.5 to L21, D25.5 to L22, D26.5 to L23, D27.5 to L24, D28.5 to L25, D29.5 to L26, D35.5 to L27, D36.5 to L28, D37.5 to L29, D3.5 to L3, D38.5 to L30, D39.5 to L31, D40.5 to L32, D42.5 to L33, D43.5 to L34, D44.5 to L35, D45.5 to L36, D46.5 to L37, D47.5 to L38, D49.5 to L39, D4.5 to L4, D50.5 to L40, D51.5 to L41, D52.5 to L42, D53.5 to L43, D54.5 to L44, D56.5 to L45, D57.5 to L46, D58.5 to L47, D59.5 to L48, D60.5 to L49, D5.5 to L5, D61.5 to L50, D62.5 to L51, D63.5 to L52, D6.5 to L6, D8.5 to L7, D9.5 to L8, D10.5 to L9, SW17 to SW10, SW18 to SW11, SW19 to SW12, SW28 to SW13, SW29 to SW14, SW30 to SW15, SW31 to SW16, SW32 to SW17, SW33 to SW18, SW7 to SW19, SW43 to SW21, SW44 to SW22, SW45 to SW23, SW46 to SW24, SW8 to SW27, SW9 to SW28, SW10 to SW29, SW11 to SW30, SW12 to SW31, SW21 to SW33, SW22 to SW34, SW23 to SW35, SW24 to SW36, SW25 to SW37, SW26 to SW38, SW35 to SW39, SW36 to SW40, SW37 to SW41, SW38 to SW42, SW39 to SW43, SW40 to SW44, SW48 to SW45, SW49 to SW46, SW50 to SW47, SW51 to SW48, SW52 to SW49, SW27 to SW50, SW14 to SW7, SW15 to SW8, SW16 to SW9
Connections:
- net L_RGB: now also U1.1 (GPIO0); no longer U1.20 (GPIO15)
- net L_VBUS: now also C46.1, C52.1, C53.1, C54.1, C55.1; no longer L1.1 (VDD), L10.1 (VDD), L11.1 (VDD), L12.1 (VDD), L13.1 (VDD), L14.1 (VDD), L15.1 (VDD), L16.1 (VDD), L17.1 (VDD), L18.1 (VDD), L19.1 (VDD), L2.1 (VDD), L20.1 (VDD), L21.1 (VDD), L22.1 (VDD), L23.1 (VDD), L24.1 (VDD), L25.1 (VDD), L26.1 (VDD), L3.1 (VDD), L4.1 (VDD), L5.1 (VDD), L6.1 (VDD), L7.1 (VDD), L8.1 (VDD), L9.1 (VDD)
- net R_C10: now also SW31.1, SW37.1, SW43.1, SW49.1; no longer SW30.1, SW36.1, SW42.1, SW48.1
- net R_C11: now also SW32.1, SW38.1, SW44.1, SW50.1; no longer SW31.1, SW37.1, SW43.1, SW49.1
- net R_C12: no longer SW32.1, SW38.1, SW44.1, SW50.1
- net R_C7: now also SW28.1, SW34.1, SW40.1, SW46.1, SW52.1; no longer SW27.1, SW33.1, SW39.1, SW45.1, SW51.1
- net R_C8: now also SW29.1, SW35.1, SW41.1, SW47.1; no longer SW28.1, SW34.1, SW40.1, SW46.1, SW52.1
- net R_C9: now also SW30.1, SW36.1, SW42.1, SW48.1; no longer SW29.1, SW35.1, SW41.1, SW47.1
- net R_RGB: now also U2.1 (GPIO0); no longer U2.20 (GPIO15)
- net R_VBUS: now also C47.1, C48.1, C49.1, C50.1, C51.1; no longer L27.1 (VDD), L28.1 (VDD), L29.1 (VDD), L30.1 (VDD), L31.1 (VDD), L32.1 (VDD), L33.1 (VDD), L34.1 (VDD), L35.1 (VDD), L36.1 (VDD), L37.1 (VDD), L38.1 (VDD), L39.1 (VDD), L40.1 (VDD), L41.1 (VDD), L42.1 (VDD), L43.1 (VDD), L44.1 (VDD), L45.1 (VDD), L46.1 (VDD), L47.1 (VDD), L48.1 (VDD), L49.1 (VDD), L50.1 (VDD), L51.1 (VDD), L52.1 (VDD)
- net at L19.4 (DIN): now also C45.1; no longer L18.2 (DOUT)
- new net: C11.1, C54.2, L13.1 (VDD)
- new net: C1.1, C52.2, L1.1 (VDD)
- new net: C33.1, C49.2, L39.1 (VDD)
- new net: C21.1, C46.2, L25.1 (VDD)
- new net: C34.2, C35.1, L41.1 (VDD)
- new net: C35.2, C36.1, L42.1 (VDD)
- new net: C5.2, L6.1 (VDD)
- new net: C19.2, C20.1, L23.1 (VDD)
- new net: C1.2, C2.1, L2.1 (VDD)
- new net: C12.2, C13.1, L15.1 (VDD)
- new net: C13.2, C14.1, L16.1 (VDD)
- new net: C2.2, C3.1, L3.1 (VDD)
- new net: C3.2, C4.1, L4.1 (VDD)
- new net: C26.2, C27.1, L31.1 (VDD)
- new net: C27.2, L32.1 (VDD)
- new net: C24.2, C25.1, L29.1 (VDD)
- new net: C25.2, C26.1, L30.1 (VDD)
- new net: C23.2, C24.1, L28.1 (VDD)
- new net: C14.2, C15.1, L17.1 (VDD)
- new net: C15.2, L18.1 (VDD)
- new net: C43.1, C47.2, L51.1 (VDD)
- new net: C43.2, L52.1 (VDD)
- new net: C30.2, C31.1, L36.1 (VDD)
- new net: C31.2, C32.1, L37.1 (VDD)
- new net: C17.2, C18.1, L21.1 (VDD)
- new net: C18.2, C19.1, L22.1 (VDD)
- new net: C53.2, C6.1, L7.1 (VDD)
- new net: C6.2, C7.1, L8.1 (VDD)
- new net: C8.2, C9.1, L10.1 (VDD)
- new net: C33.2, C34.1, L40.1 (VDD)
- new net: C28.2, C29.1, L34.1 (VDD)
- new net: C10.1, C9.2, L11.1 (VDD)
- new net: C10.2, L12.1 (VDD)
- new net: C11.2, C12.1, L14.1 (VDD)
- new net: C20.2, L24.1 (VDD)
- new net: C23.1, C51.2, L27.1 (VDD)
- new net: C37.2, L44.1 (VDD)
- new net: C4.2, C5.1, L5.1 (VDD)
- new net: C7.2, C8.1, L9.1 (VDD)
- new net: C32.2, L38.1 (VDD)
- new net: C16.1, C55.2, L19.1 (VDD)
- new net: C16.2, C17.1, L20.1 (VDD)
- new net: C41.2, C42.1, L49.1 (VDD)
- new net: C38.1, C48.2, L45.1 (VDD)
- new net: C38.2, C39.1, L46.1 (VDD)
- new net: C29.2, C30.1, L35.1 (VDD)
- new net: C45.2, L18.2 (DOUT)
- new net: C39.2, C40.1, L47.1 (VDD)
- new net: C40.2, C41.1, L48.1 (VDD)
- new net: C42.2, L50.1 (VDD)
- new net: C21.2, L26.1 (VDD)
- new net: C36.2, C37.1, L43.1 (VDD)
- new net: C28.1, C50.2, L33.1 (VDD)
- new net R_C6: SW27.1, SW33.1, SW39.1, SW45.1, SW51.1
Other:
- note added: "https://www.mouser.com/ProductDetail/Samsung-Electro-Mechanics/CL21A107MQYNNWE?qs=sGAEpiMZZMsh%252B1woXyUXj7hTFrnMyX907rJbWHkejgM%3D"
- note added: "use these 100 uf capacitors:"

Commit message: PCB Done!
Parts:
- removed C25, C26, C45: C 100uf, Capacitor_SMD:C_0805_2012Metric_Pad1.18x1.45mm_HandSolder, symbol Device:C
- added C4, C6: C 100uf, Capacitor_SMD:C_0805_2012Metric_Pad1.18x1.45mm_HandSolder, symbol Device:C
- renumbered C52 to C1, C23 to C10, C53 to C11, C32 to C12, C7 to C13, C30 to C14, C8 to C15, C29 to C16, C6 to C17, C31 to C18, C5 to C19, C27 to C2, C51 to C20, C9 to C21, C28 to C22, C12 to C23, C35 to C24, C54 to C25, C37 to C26, C13 to C27, C34 to C28, C11 to C29, C2 to C3, C36 to C30, C10 to C31, C50 to C32, C14 to C33, C33 to C34, C17 to C35, C40 to C36, C55 to C37, C42 to C38, C18 to C39, C39 to C40, C16 to C41, C41 to C42, C15 to C43, C49 to C44, C19 to C45, C38 to C46, C20 to C47, C46 to C49, C1 to C5, C43 to C50, C21 to C51, C47 to C52, C3 to C7, C24 to C8, C4 to C9, D28 to D10, D7 to D11, D38 to D12, D9 to D13, D36 to D14, D10 to D15, D35 to D16, D8 to D17, D37 to D18, D6 to D19, D32 to D2, D27 to D20, D11 to D21, D34 to D22, D15 to D23, D42 to D24, D13 to D25, D44 to D26, D16 to D27, D41 to D28, D14 to D29, D43 to D30, D12 to D31, D33 to D32, D17 to D33, D40 to D34, D21 to D35, D48 to D36, D19 to D37, D50 to D38, D22 to D39, D30 to D4, D47 to D40, D20 to D41, D49 to D42, D18 to D43, D39 to D44, D23 to D45, D24 to D47, D45 to D48, D25 to D49, D2 to D5, D52 to D50, D26 to D51, D51 to D52, D31 to D6, D4 to D7, D29 to D8, D5 to D9, L28 to L10, L7 to L11, L38 to L12, L9 to L13, L36 to L14, L10 to L15, L35 to L16, L8 to L17, L37 to L18, L6 to L19, L32 to L2, L27 to L20, L11 to L21, L34 to L22, L15 to L23, L42 to L24, L13 to L25, L44 to L26, L16 to L27, L41 to L28, L14 to L29, L43 to L30, L12 to L31, L33 to L32, L17 to L33, L40 to L34, L21 to L35, L48 to L36, L19 to L37, L50 to L38, L22 to L39, L30 to L4, L47 to L40, L20 to L41, L49 to L42, L18 to L43, L39 to L44, L23 to L45, L24 to L47, L45 to L48, L25 to L49, L2 to L5, L52 to L50, L26 to L51, L51 to L52, L31 to L6, L4 to L7, L29 to L8, L5 to L9, SW28 to SW10, SW7 to SW11, SW38 to SW12, SW9 to SW13, SW36 to SW14, SW10 to SW15, SW35 to SW16, SW8 to SW17, SW37 to SW18, SW6 to SW19, SW32 to SW2, SW27 to SW20, SW11 to SW21, SW34 to SW22, SW15 to SW23, SW42 to SW24, SW13 to SW25, SW44 to SW26, SW16 to SW27, SW41 to SW28, SW14 to SW29, SW43 to SW30, SW12 to SW31, SW33 to SW32, SW17 to SW33, SW40 to SW34, SW21 to SW35, SW48 to SW36, SW19 to SW37, SW50 to SW38, SW22 to SW39, SW30 to SW4, SW47 to SW40, SW20 to SW41, SW49 to SW42, SW18 to SW43, SW39 to SW44, SW23 to SW45, SW24 to SW47, SW45 to SW48, SW25 to SW49, SW2 to SW5, SW52 to SW50, SW26 to SW51, SW51 to SW52, SW31 to SW6, SW4 to SW7, SW29 to SW8, SW5 to SW9
Connections:
- net L_GND is gone; now on net GND: U1.42 (GND)
- net L_R0: now also U1.27 (GPIO21); no longer U1.22 (GPIO17)
- net L_R1: now also U1.26 (GPIO20); no longer U1.24 (GPIO18)
- net L_R3: now also U1.24 (GPIO18); no longer U1.26 (GPIO20)
- net L_R4: now also U1.22 (GPIO17); no longer U1.27 (GPIO21)
- net L_TX: no longer J2.3 (R1)
- net R_C6: now also U2.9 (GPIO6)
- net R_R0: now also U2.27 (GPIO21); no longer U2.22 (GPIO17)
- net R_R1: now also U2.26 (GPIO20); no longer U2.24 (GPIO18)
- net R_R3: now also U2.24 (GPIO18); no longer U2.26 (GPIO20)
- net R_R4: now also U2.22 (GPIO17); no longer U2.27 (GPIO21)
- net R_TX: now also J2.3 (R1)
- net at C2.1, L6.1 (VDD): now also C6.2
- net at C8.2, L8.1 (VDD): now also C4.1
- net at L4.1 (VDD): now also C4.2, C6.1
- net at L37.4 (DIN): now also L43.2 (DOUT)
- net R_C12: no longer names the net of U2.16 (GPIO12)
- no-connect marks 42 -> 41
Other:
- moved on the sheet: C8

Commit message: Neopixels power fixed
Parts:
- removed C10, C18, C19, C21, C22, C23, C24, C25, C26, C27, C28, C29, C3, C30, C31, C32, C33, C34, C35, C36, C37, C38, C39, C40, C41, C42, C43, C44, C45, C46, C47, C48, C49, C50, C51: C 100uf, Capacitor_SMD:C_0805_2012Metric_Pad1.18x1.45mm_HandSolder, symbol Device:C
- added C11: C 10uf, Capacitor_SMD:C_0805_2012Metric_Pad1.18x1.45mm_HandSolder, symbol Device:C
- C1, C12, C13, C14, C15, C16, C17, C2, C4, C5, C6, C7, C8, C9: value C 100uf -> C 10uf
- C10: renamed from C20; value C 100uf -> C 10uf
- C18: renamed from C52; value C 100uf -> C 10uf
- C3: renamed from C11; value C 100uf -> C 10uf
Connections:
- net GND: now also C1.1, C10.1, C12.1, C13.1, C14.1, C15.1, C16.1, C17.1, C18.1, C2.1, C3.1, C4.1, C5.1, C6.1, C7.1, C8.1, C9.1, C11.1
- net L_VBUS: now also C1.2, C2.2, C3.2, C4.2, C5.2, C6.2, C7.2, C8.2, C9.2, L1.1 (VDD), L11.1 (VDD), L13.1 (VDD), L15.1 (VDD), L17.1 (VDD), L19.1 (VDD), L21.1 (VDD), L23.1 (VDD), L25.1 (VDD), L27.1 (VDD), L29.1 (VDD), L3.1 (VDD), L31.1 (VDD), L33.1 (VDD), L35.1 (VDD), L37.1 (VDD), L39.1 (VDD), L41.1 (VDD), L43.1 (VDD), L45.1 (VDD), L47.1 (VDD), L49.1 (VDD), L5.1 (VDD), L51.1 (VDD), L7.1 (VDD), L9.1 (VDD); no longer C1.1, C3.1
- net R_VBUS: now also C10.2, C12.2, C13.2, C14.2, C15.2, C16.2, C17.2, C18.2, L10.1 (VDD), L12.1 (VDD), L14.1 (VDD), L16.1 (VDD), L18.1 (VDD), L2.1 (VDD), L20.1 (VDD), L22.1 (VDD), L24.1 (VDD), L26.1 (VDD), L28.1 (VDD), L30.1 (VDD), L32.1 (VDD), L34.1 (VDD), L36.1 (VDD), L38.1 (VDD), L4.1 (VDD), L40.1 (VDD), L42.1 (VDD), L44.1 (VDD), L46.1 (VDD), L48.1 (VDD), L50.1 (VDD), L52.1 (VDD), L6.1 (VDD), L8.1 (VDD), C11.2; no longer C10.1, C18.1
Other:
- note added: "https://www.digikey.com/en/products/detail/murata-electronics/GRM21BR61C106KE15K/2546903"
- note added: "use these 10 uf capacitors:"
- note removed: "https://www.mouser.com/ProductDetail/Samsung-Electro-Mechanics/CL21A107MQYNNWE?qs=sGAEpiMZZMsh%252B1woXyUXj7hTFrnMyX907rJbWHkejgM%3D"
- note removed: "use these 100 uf capacitors:"
- moved on the sheet: C1, C10, C18, C3
